File: KiCad files/LED_Cube_5X5X5/LED_Cube_5X5X5.kicad_pcb (KiCad board)
At the start: 2 copper layers, 100 x 100 mm, 66 parts, among them J1 Barrel_Jack_MountingPin, J2 USBASP, J3 CON1, J4 CON2, J5 CON3, Q1 BC337, Q2 BC337, Q3 BC337, Q4 BC337, Q5 BC337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

Commit message: test
Other:
- net class Default removed
